Commit message: Update wx250.urdf.xacro

File: robots/wx250_description/urdf/wx250.urdf.xacro (robot description, xacro)
@@ -9,337 +9,232 @@
   <xacro:arg name="external_urdf_loc" default=""/>
   <xacro:arg name="load_gazebo_configs" default="false"/>
-  <xacro:property name="urdf_loc" value="$(arg external_urdf_loc)"/>
-  <xacro:property name="pi_offset" value="0.00001"/>
-  <xacro:if value="$(arg load_gazebo_configs)">
-    <xacro:include filename="$(find interbotix_xsarm_gazebo)/config/interbotix_texture.gazebo"/>
-  </xacro:if>
-  <material name="interbotix_black">
-    <texture filename="package://interbotix_xsarm_descriptions/meshes/interbotix_black.png"/>
-  </material>
-  <xacro:if value="$(arg use_world_frame)">
-    <link name="world"/>
-    <joint name="fixed" type="fixed">
-      <parent link="world"/>
-      <child link="$(arg robot_name)/$(arg base_link_frame)"/>
-    </joint>
-  </xacro:if>
-  <link name="$(arg robot_name)/$(arg base_link_frame)">
-    <visual>
-      <origin rpy="0 0 ${pi/2}" xyz="0 0 0"/>
-      <geometry>
-        <mesh filename="package://interbotix_xsarm_descriptions/meshes/wx250_meshes/wx250_1_base.stl" scale="0.001 0.001 0.001"/>
-      </geometry>
-      <material name="interbotix_black"/>
-    </visual>
-    <collision>
-      <origin rpy="0 0 ${pi/2}" xyz="0 0 0"/>
-      <geometry>
-        <mesh filename="package://interbotix_xsarm_descriptions/meshes/wx250_meshes/wx250_1_base.stl" scale="0.001 0.001 0.001"/>
-      </geometry>
-    </collision>
-    <inertial>
-      <origin rpy="0 0 ${pi/2}" xyz="-0.0380446000 0.0006138920 0.0193354000"/>
-      <mass value="0.538736" />
-      <inertia ixx="0.0021150000" iyy="0.0006921000" izz="0.0025240000" ixy="-0.0000163500" ixz="0.0000006998" iyz="0.0000464200" />
-    </inertial>
-  </link>
-  <joint name="waist" type="revolute">
-    <axis xyz="0 0 1"/>
-    <limit effort="10" lower="${-pi + pi_offset}" upper="${pi - pi_offset}" velocity="${pi}"/>
-    <origin rpy="0 0 0" xyz="0 0 0.072"/>
-    <parent link="$(arg robot_name)/$(arg base_link_frame)"/>
-    <child link="$(arg robot_name)/shoulder_link"/>
-    <dynamics friction="0.1"/>
-  </joint>
-  <transmission name="trans_waist">
-    <type>transmission_interface/SimpleTransmission</type>
-    <joint name="waist">
-      <hardwareInterface>hardware_interface/EffortJointInterface</hardwareInterface>
-    </joint>
-    <actuator name="waist_motor">
-      <mechanicalReduction>1</mechanicalReduction>
-    </actuator>
-  </transmission>
-  <link name="$(arg robot_name)/shoulder_link">
-    <visual>
-      <origin rpy="0 0 ${pi/2}" xyz="0 0 -0.003"/>
-      <geometry>
-        <mesh filename="package://interbotix_xsarm_descriptions/meshes/wx250_meshes/wx250_2_shoulder.stl" scale="0.001 0.001 0.001"/>
-      </geometry>
-      <material name="interbotix_black"/>
-    </visual>
-    <collision>
-      <origin rpy="0 0 ${pi/2}" xyz="0 0 -0.003"/>
-      <geometry>
-        <mesh filename="package://interbotix_xsarm_descriptions/meshes/wx250_meshes/wx250_2_shoulder.stl" scale="0.001 0.001 0.001"/>
-      </geometry>
-    </collision>
-    <inertial>
-      <origin rpy="0 0 ${pi/2}" xyz="0.0000223482 0.0000414609 0.0066287000"/>
-      <mass value="0.480879" />
-      <inertia ixx="0.0003790000" iyy="0.0005557000" izz="0.0005889000" ixy="0.0000000022" ixz="-0.0000003561" iyz="0.0000012245" />
-    </inertial>
-  </link>
-  <joint name="shoulder" type="revolute">
-    <axis xyz="0 1 0"/>
-    <limit effort="20" lower="${radians(-108)}" upper="${radians(114)}" velocity="${pi}"/>
-    <origin rpy="0 0 0" xyz="0 0 0.03865"/>
-    <parent link="$(arg robot_name)/shoulder_link"/>
-    <child link="$(arg robot_name)/upper_arm_link"/>
-    <dynamics friction="0.1"/>
-  </joint>
-  <transmission name="trans_shoulder">
-    <type>transmission_interface/SimpleTransmission</type>
-    <joint name="shoulder">
-      <hardwareInterface>hardware_interface/EffortJointInterface</hardwareInterface>
-    </joint>
-    <actuator name="shoulder_motor">
-      <mechanicalReduction>1</mechanicalReduction>
-    </actuator>
-  </transmission>
-  <link name="$(arg robot_name)/upper_arm_link">
-    <visual>
-      <origin rpy="0 0 ${pi/2}" xyz="0 0 0"/>
-      <geometry>
-        <mesh filename="package://interbotix_xsarm_descriptions/meshes/wx250_meshes/wx250_3_upper_arm.stl" scale="0.001 0.001 0.001"/>
-      </geometry>
-      <material name="interbotix_black"/>
-    </visual>
-    <collision>
-      <origin rpy="0 0 ${pi/2}" xyz="0 0 0"/>
-      <geometry>
-        <mesh filename="package://interbotix_xsarm_descriptions/meshes/wx250_meshes/wx250_3_upper_arm.stl" scale="0.001 0.001 0.001"/>
-      </geometry>
-    </collision>
-    <inertial>
-      <origin rpy="0 0 ${pi/2}" xyz="0.0171605000 0.0000002725 0.1913230000"/>
-      <mass value="0.430811" />
-      <inertia ixx="0.0034630000" iyy="0.0035870000" izz="0.0004566000" ixy="-0.0000000001" ixz="-0.0000000002" iyz="0.0004272000" />
-    </inertial>
-  </link>
-  <joint name="elbow" type="revolute">
-    <axis xyz="0 1 0"/>
-    <limit effort="15" lower="${radians(-123)}" upper="${radians(92)}" velocity="${pi}"/>
-    <origin rpy="0 0 0" xyz="0.04975 0 0.25"/>
-    <parent link="$(arg robot_name)/upper_arm_link"/>
-    <child link="$(arg robot_name)/forearm_link"/>
-    <dynamics friction="0.1"/>
-  </joint>
-  <transmission name="trans_elbow">
-    <type>transmission_interface/SimpleTransmission</type>
-    <joint name="elbow">
-      <hardwareInterface>hardware_interface/EffortJointInterface</hardwareInterface>
-    </joint>
-    <actuator name="elbow_motor">
-      <mechanicalReduction>1</mechanicalReduction>
-    </actuator>
-  </transmission>
-  <link name="$(arg robot_name)/forearm_link">
-    <visual>
-      <origin rpy="0 0 ${pi/2}" xyz="0 0 0"/>
-      <geometry>
-        <mesh filename="package://interbotix_xsarm_descriptions/meshes/wx250_meshes/wx250_4_forearm.stl" scale="0.001 0.001 0.001"/>
-      </geometry>
-      <material name="interbotix_black"/>
-    </visual>
-    <collision>
-      <origin rpy="0 0 ${pi/2}" xyz="0 0 0"/>
-      <geometry>
-        <mesh filename="package://interbotix_xsarm_descriptions/meshes/wx250_meshes/wx250_4_forearm.stl" scale="0.001 0.001 0.001"/>
-      </geometry>
-    </collision>
-    <inertial>
-      <origin rpy="0 0 ${pi/2}" xyz="0.1534230000 -0.0001179685 -0.0004390000"/>
-      <mass value="0.297673" />
-      <inertia ixx="0.0021760000" iyy="0.0000575700" izz="0.0021860000" ixy="-0.0000030658" ixz="0.0000000000" iyz="0.0000000000" />
-    </inertial>
-  </link>
- <joint name="wrist_angle" type="revolute">
-    <axis xyz="0 1 0"/>
-    <limit effort="5" lower="${radians(-100)}" upper="${radians(123)}" velocity="${pi}"/>
-    <origin rpy="0 0 0" xyz="0.25 0 0"/>
-    <parent link="$(arg robot_name)/forearm_link"/>
-    <child link="$(arg robot_name)/wrist_link"/>
-    <dynamics friction="0.1"/>
-  </joint>
-  <transmission name="trans_wrist_angle">
-    <type>transmission_interface/SimpleTransmission</type>
-    <joint name="wrist_angle">
-      <hardwareInterface>hardware_interface/EffortJointInterface</hardwareInterface>
-    </joint>
-    <actuator name="wrist_angle_motor">
-      <mechanicalReduction>1</mechanicalReduction>
-    </actuator>
-  </transmission>
-  <link name="$(arg robot_name)/wrist_link">
-    <visual>
-      <origin rpy="0 0 ${pi/2}" xyz="0 0 0"/>
-      <geometry>
-        <mesh filename="package://interbotix_xsarm_descriptions/meshes/wx250_meshes/wx250_5_wrist.stl" scale="0.001 0.001 0.001"/>
-      </geometry>
-      <material name="interbotix_black"/>
-    </visual>
-    <collision>
-      <origin rpy="0 0 ${pi/2}" xyz="0 0 0"/>
-      <geometry>
-        <mesh filename="package://interbotix_xsarm_descriptions/meshes/wx250_meshes/wx250_5_wrist.stl" scale="0.001 0.001 0.001"/>
-      </geometry>
-    </collision>
-    <inertial>
-      <origin rpy="0 0 ${pi/2}" xyz="0.0423600000 -0.0000106630 0.0105770000"/>
-      <mass value="0.084957" />
-      <inertia ixx="0.0000308200" iyy="0.0000282200" izz="0.0000315200" ixy="0.0000000191" ixz="0.0000000023" iyz="0.0000025481" />
-    </inertial>
-  </link>
-  <joint name="wrist_rotate" type="revolute">
-    <axis xyz="1 0 0"/>
-    <limit effort="1" lower="${-pi + pi_offset}" upper="${pi - pi_offset}" velocity="${pi}"/>
-    <origin rpy="0 0 0" xyz="0.065 0 0"/>
-    <parent link="$(arg robot_name)/wrist_link"/>
-    <child link="$(arg robot_name)/gripper_link"/>
-    <dynamics friction="0.1"/>
-  </joint>
-  <transmission name="trans_wrist_rotate">
-    <type>transmission_interface/SimpleTransmission</type>
-    <joint name="wrist_rotate">
-      <hardwareInterface>hardware_interface/EffortJointInterface</hardwareInterface>
-    </joint>
-    <actuator name="wrist_rotate_motor">
-      <mechanicalReduction>1</mechanicalReduction>
-    </actuator>
-  </transmission>
-  <link name="$(arg robot_name)/gripper_link">
-    <visual>
-      <origin rpy="0 0 ${pi/2}" xyz="-0.02 0 0"/>
-      <geometry>
-        <mesh filename="package://interbotix_xsarm_descriptions/meshes/wx250_meshes/wx250_6_gripper.stl" scale="0.001 0.001 0.001"/>
-      </geometry>
-      <material name="interbotix_black"/>
-    </visual>
-    <collision>
-      <origin rpy="0 0 ${pi/2}" xyz="-0.02 0 0"/>
-      <geometry>
-        <mesh filename="package://interbotix_xsarm_descriptions/meshes/wx250_meshes/wx250_6_gripper.stl" scale="0.001 0.001 0.001"/>
-      </geometry>
-    </collision>
-    <inertial>
-      <origin rpy="0 0 ${pi/2}" xyz="0.0216310000 0.0000002516 0.0114100000"/>
-      <mass value="0.072885" />
-      <inertia ixx="0.0000253700" iyy="0.0000183600" izz="0.0000167400" ixy="0.0000000000" ixz="0.0000000000" iyz="0.0000004340" />
-    </inertial>
-  </link>
-  <joint name="ee_arm" type="fixed">
-    <axis xyz="1 0 0"/>
-    <origin rpy="0 0 0" xyz="0.043 0 0"/>
-    <parent link="$(arg robot_name)/gripper_link"/>
-    <child link="$(arg robot_name)/ee_arm_link"/>
-  </joint>
-  <link name="$(arg robot_name)/ee_arm_link">
-    <inertial>
-      <mass value="0.001" />
-      <inertia ixx="0.001" iyy="0.001" izz="0.001" ixy="0" ixz="0" iyz="0" />
-    </inertial>
-  </link>
-  <joint name="gripper" type="continuous">
-    <axis xyz="1 0 0"/>
-    <limit effort="1" velocity="${pi}"/>
-    <origin rpy="0 0 0" xyz="0.0055 0 0"/>
-    <parent link="$(arg robot_name)/ee_arm_link"/>
-    <child link="$(arg robot_name)/gripper_prop_link"/>
-    <dynamics friction="0.1"/>
-  </joint>
-  <transmission name="trans_gripper">
-    <type>transmission_interface/SimpleTransmission</type>
-    <joint name="gripper">
-      <hardwareInterface>hardware_interface/EffortJointInterface</hardwareInterface>
-    </joint>
-    <actuator name="gripper_motor">
-      <mechanicalReduction>1</mechanicalReduction>
-    </actuator>
-  </transmission>
-  <link name="$(arg robot_name)/gripper_prop_link">
-    <visual>
-      <origin rpy="0 0 ${pi/2}" xyz="-0.0685 0 0"/>
-      <geometry>
-        <mesh filename="package://interbotix_xsarm_descriptions/meshes/wx250_meshes/wx250_7_gripper_prop.stl" scale="0.001 0.001 0.001"/>
-      </geometry>
-      <material name="interbotix_black"/>
-    </visual>
-    <collision>
-      <origin rpy="0 0 ${pi/2}" xyz="-0.0685 0 0"/>
-      <geometry>
-        <mesh filename="package://interbotix_xsarm_descriptions/meshes/wx250_meshes/wx250_7_gripper_prop.stl" scale="0.001 0.001 0.001"/>
-      </geometry>
-    </collision>
-    <inertial>
-      <origin rpy="0 0 ${pi/2}" xyz="0.0008460000 -0.0000016817 0.0000420000"/>
-      <mass value="0.00434" />
-      <inertia ixx="0.0000005923" iyy="0.0000011156" izz="0.0000005743" ixy="0.0000000000" ixz="0.0000003195" iyz="-0.0000000004" />
-    </inertial>
-  </link>
-  <!-- If the AR tag is being used, then add the AR tag mount -->
-  <xacro:if value="$(arg show_ar_tag)">
-    <joint name="ar_tag" type="fixed">
-      <axis xyz="0 0 0"/>
-      <origin rpy="0 0 0" xyz="-0.017 0 0.04155"/>
-      <parent link="$(arg robot_name)/ee_arm_link"/>
-      <child link="$(arg robot_name)/ar_tag_link"/>
-    </joint>
-    <link name="$(arg robot_name)/ar_tag_link">
-      <visual>
-        <origin rpy="0 0 0" xyz="0 0 0"/>
-        <geometry>
-          <mesh filename="package://interbotix_xsarm_descriptions/meshes/wx250_meshes/wx250_10_ar_tag.stl" scale="0.001 0.001 0.001"/>
-        </geometry>
-        <material name="interbotix_black"/>
-      </visual>
-      <collision>
-        <origin rpy="0 0 0" xyz="0 0 0"/>
-        <geometry>
-          <mesh filename="package://interbotix_xsarm_descriptions/meshes/wx250_meshes/wx250_10_ar_tag.stl" scale="0.001 0.001 0.001"/>
-        </geometry>
-      </collision>
-      <inertial>
-        <origin rpy="0 0 0" xyz="0 0 -0.00315"/>
-        <mass value="0.016507"/>
-        <inertia ixx="0.000003084" ixy="0" ixz="0" iyy="0.000003084" iyz="0" izz="0.000006059"/>
-      </inertial>
-    </link>
-  </xacro:if>
-  <!-- If the gripper bar is being used, then also add the gripper bar -->
-  <xacro:if value="$(arg show_gripper_bar)">
-    <joint name="gripper_bar" type="fixed">
+  <xacro:macro name="wx250_robot" params="">
+    <xacro:property name="urdf_loc" value="$(arg external_urdf_loc)"/>
+    <xacro:property name="pi_offset" value="0.00001"/>
+    <xacro:if value="$(arg load_gazebo_configs)">
+      <xacro:include filename="$(find interbotix_xsarm_gazebo)/config/interbotix_texture.gazebo"/>
+    </xacro:if>
+    <material name="interbotix_black">
+      <texture filename="package://interbotix_xsarm_descriptions/meshes/interbotix_black.png"/>
+    </material>
+    <xacro:if value="$(arg use_world_frame)">
+      <link name="world"/>
+      <joint name="fixed" type="fixed">
+        <parent link="world"/>
+        <child link="$(arg robot_name)/$(arg base_link_frame)"/>
+      </joint>
+    </xacro:if>
+    <link name="$(arg robot_name)/$(arg base_link_frame)">
+      <visual>
+        <origin rpy="0 0 ${pi/2}" xyz="0 0 0"/>
+        <geometry>
+          <mesh filename="package://interbotix_xsarm_descriptions/meshes/wx250_meshes/wx250_1_base.stl" scale="0.001 0.001 0.001"/>
+        </geometry>
+        <material name="interbotix_black"/>
+      </visual>
+      <collision>
+        <origin rpy="0 0 ${pi/2}" xyz="0 0 0"/>
+        <geometry>
+          <mesh filename="package://interbotix_xsarm_descriptions/meshes/wx250_meshes/wx250_1_base.stl" scale="0.001 0.001 0.001"/>
+        </geometry>
+      </collision>
+      <inertial>
+        <origin rpy="0 0 ${pi/2}" xyz="-0.0380446000 0.0006138920 0.0193354000"/>
+        <mass value="0.538736" />
+        <inertia ixx="0.0021150000" iyy="0.0006921000" izz="0.0025240000" ixy="-0.0000163500" ixz="0.0000006998" iyz="0.0000464200" />
+      </inertial>
+    </link>
+    <joint name="waist" type="revolute">
+      <axis xyz="0 0 1"/>
+      <limit effort="10" lower="${-pi + pi_offset}" upper="${pi - pi_offset}" velocity="${pi}"/>
+      <origin rpy="0 0 0" xyz="0 0 0.072"/>
+      <parent link="$(arg robot_name)/$(arg base_link_frame)"/>
+      <child link="$(arg robot_name)/shoulder_link"/>
+      <dynamics friction="0.1"/>
+    </joint>
+    <transmission name="trans_waist">
+      <type>transmission_interface/SimpleTransmission</type>
+      <joint name="waist">
+        <hardwareInterface>hardware_interface/EffortJointInterface</hardwareInterface>
+      </joint>
+      <actuator name="waist_motor">
+        <mechanicalReduction>1</mechanicalReduction>
+      </actuator>
+    </transmission>
+    <link name="$(arg robot_name)/shoulder_link">
+      <visual>
+        <origin rpy="0 0 ${pi/2}" xyz="0 0 -0.003"/>
+        <geometry>
+          <mesh filename="package://interbotix_xsarm_descriptions/meshes/wx250_meshes/wx250_2_shoulder.stl" scale="0.001 0.001 0.001"/>
+        </geometry>
+        <material name="interbotix_black"/>
+      </visual>
+      <collision>
+        <origin rpy="0 0 ${pi/2}" xyz="0 0 -0.003"/>
+        <geometry>
+          <mesh filename="package://interbotix_xsarm_descriptions/meshes/wx250_meshes/wx250_2_shoulder.stl" scale="0.001 0.001 0.001"/>
+        </geometry>
+      </collision>
+      <inertial>
+        <origin rpy="0 0 ${pi/2}" xyz="0.0000223482 0.0000414609 0.0066287000"/>
+        <mass value="0.480879" />
+        <inertia ixx="0.0003790000" iyy="0.0005557000" izz="0.0005889000" ixy="0.0000000022" ixz="-0.0000003561" iyz="0.0000012245" />
+      </inertial>
+    </link>
+    <joint name="shoulder" type="revolute">
+      <axis xyz="0 1 0"/>
+      <limit effort="20" lower="${radians(-108)}" upper="${radians(114)}" velocity="${pi}"/>
+      <origin rpy="0 0 0" xyz="0 0 0.03865"/>
+      <parent link="$(arg robot_name)/shoulder_link"/>
+      <child link="$(arg robot_name)/upper_arm_link"/>
+      <dynamics friction="0.1"/>
+    </joint>
+    <transmission name="trans_shoulder">
+      <type>transmission_interface/SimpleTransmission</type>
+      <joint name="shoulder">
+        <hardwareInterface>hardware_interface/EffortJointInterface</hardwareInterface>
+      </joint>
+      <actuator name="shoulder_motor">
+        <mechanicalReduction>1</mechanicalReduction>
+      </actuator>
+    </transmission>
+    <link name="$(arg robot_name)/upper_arm_link">
+      <visual>
+        <origin rpy="0 0 ${pi/2}" xyz="0 0 0"/>
+        <geometry>
+          <mesh filename="package://interbotix_xsarm_descriptions/meshes/wx250_meshes/wx250_3_upper_arm.stl" scale="0.001 0.001 0.001"/>
+        </geometry>
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