Commit message: Update wx250.urdf.xacro

File: robots/wx250_description/urdf/wx250.urdf.xacro (robot description, xacro)
@@ -13,8 +13,8 @@
     <xacro:property name="pi_offset" value="0.00001"/>
     <xacro:if value="$(arg load_gazebo_configs)">
-      <xacro:include filename="$(find interbotix_xsarm_gazebo)/config/interbotix_texture.gazebo"/>
+      <xacro:include filename="$(find wx250_description)/config/interbotix_texture.gazebo"/>
     </xacro:if>
     <material name="interbotix_black">
-      <texture filename="package://interbotix_xsarm_descriptions/meshes/interbotix_black.png"/>
+      <texture filename="package://wx250_description/meshes/interbotix_black.png"/>
     </material>
     <xacro:if value="$(arg use_world_frame)">
@@ -29,12 +29,12 @@
         <origin rpy="0 0 ${pi/2}" xyz="0 0 0"/>
         <geometry>
-          <mesh filename="package://interbotix_xsarm_descriptions/meshes/wx250_meshes/wx250_1_base.stl" scale="0.001 0.001 0.001"/>
-        </geometry>
-        <material name="interbotix_black"/>
-      </visual>
-      <collision>
-        <origin rpy="0 0 ${pi/2}" xyz="0 0 0"/>
-        <geometry>
-          <mesh filename="package://interbotix_xsarm_descriptions/meshes/wx250_meshes/wx250_1_base.stl" scale="0.001 0.001 0.001"/>
+          <mesh filename="package://wx250_description/meshes/wx250_1_base.stl" scale="0.001 0.001 0.001"/>
+        </geometry>
+        <material name="interbotix_black"/>
+      </visual>
+      <collision>
+        <origin rpy="0 0 ${pi/2}" xyz="0 0 0"/>
+        <geometry>
+          <mesh filename="package://wx250_description/meshes/wx250_1_base.stl" scale="0.001 0.001 0.001"/>
         </geometry>
       </collision>
@@ -66,5 +66,5 @@
         <origin rpy="0 0 ${pi/2}" xyz="0 0 -0.003"/>
         <geometry>
-          <mesh filename="package://interbotix_xsarm_descriptions/meshes/wx250_meshes/wx250_2_shoulder.stl" scale="0.001 0.001 0.001"/>
+          <mesh filename="package://wx250_description/meshes/wx250_2_shoulder.stl" scale="0.001 0.001 0.001"/>
         </geometry>
         <material name="interbotix_black"/>
@@ -73,5 +73,5 @@
         <origin rpy="0 0 ${pi/2}" xyz="0 0 -0.003"/>
         <geometry>
-          <mesh filename="package://interbotix_xsarm_descriptions/meshes/wx250_meshes/wx250_2_shoulder.stl" scale="0.001 0.001 0.001"/>
+          <mesh filename="package://wx250_description/meshes/wx250_2_shoulder.stl" scale="0.001 0.001 0.001"/>
         </geometry>
       </collision>
@@ -103,12 +103,12 @@
         <origin rpy="0 0 ${pi/2}" xyz="0 0 0"/>
         <geometry>
-          <mesh filename="package://interbotix_xsarm_descriptions/meshes/wx250_meshes/wx250_3_upper_arm.stl" scale="0.001 0.001 0.001"/>
-        </geometry>
-        <material name="interbotix_black"/>
-      </visual>
-      <collision>
-        <origin rpy="0 0 ${pi/2}" xyz="0 0 0"/>
-        <geometry>
-          <mesh filename="package://interbotix_xsarm_descriptions/meshes/wx250_meshes/wx250_3_upper_arm.stl" scale="0.001 0.001 0.001"/>
+          <mesh filename="package://wx250_description/meshes/wx250_3_upper_arm.stl" scale="0.001 0.001 0.001"/>
+        </geometry>
+        <material name="interbotix_black"/>
+      </visual>
+      <collision>
+        <origin rpy="0 0 ${pi/2}" xyz="0 0 0"/>
+        <geometry>
+          <mesh filename="package://wx250_description/meshes/wx250_3_upper_arm.stl" scale="0.001 0.001 0.001"/>
         </geometry>
       </collision>
@@ -140,12 +140,12 @@
         <origin rpy="0 0 ${pi/2}" xyz="0 0 0"/>
         <geometry>
-          <mesh filename="package://interbotix_xsarm_descriptions/meshes/wx250_meshes/wx250_4_forearm.stl" scale="0.001 0.001 0.001"/>
-        </geometry>
-        <material name="interbotix_black"/>
-      </visual>
-      <collision>
-        <origin rpy="0 0 ${pi/2}" xyz="0 0 0"/>
-        <geometry>
-          <mesh filename="package://interbotix_xsarm_descriptions/meshes/wx250_meshes/wx250_4_forearm.stl" scale="0.001 0.001 0.001"/>
+          <mesh filename="package://wx250_description/meshes/wx250_4_forearm.stl" scale="0.001 0.001 0.001"/>
+        </geometry>
+        <material name="interbotix_black"/>
+      </visual>
+      <collision>
+        <origin rpy="0 0 ${pi/2}" xyz="0 0 0"/>
+        <geometry>
+          <mesh filename="package://wx250_description/meshes/wx250_4_forearm.stl" scale="0.001 0.001 0.001"/>
         </geometry>
       </collision>
@@ -177,12 +177,12 @@
         <origin rpy="0 0 ${pi/2}" xyz="0 0 0"/>
         <geometry>
-          <mesh filename="package://interbotix_xsarm_descriptions/meshes/wx250_meshes/wx250_5_wrist.stl" scale="0.001 0.001 0.001"/>
-        </geometry>
-        <material name="interbotix_black"/>
-      </visual>
-      <collision>
-        <origin rpy="0 0 ${pi/2}" xyz="0 0 0"/>
-        <geometry>
-          <mesh filename="package://interbotix_xsarm_descriptions/meshes/wx250_meshes/wx250_5_wrist.stl" scale="0.001 0.001 0.001"/>
+          <mesh filename="package://wx250_description/meshes/wx250_5_wrist.stl" scale="0.001 0.001 0.001"/>
+        </geometry>
+        <material name="interbotix_black"/>
+      </visual>
+      <collision>
+        <origin rpy="0 0 ${pi/2}" xyz="0 0 0"/>
+        <geometry>
+          <mesh filename="package://wx250_description/meshes/wx250_5_wrist.stl" scale="0.001 0.001 0.001"/>
         </geometry>
       </collision>
@@ -214,5 +214,5 @@
         <origin rpy="0 0 ${pi/2}" xyz="-0.02 0 0"/>
         <geometry>
-          <mesh filename="package://interbotix_xsarm_descriptions/meshes/wx250_meshes/wx250_6_gripper.stl" scale="0.001 0.001 0.001"/>
+          <mesh filename="package://wx250_description/meshes/wx250_6_gripper.stl" scale="0.001 0.001 0.001"/>
         </geometry>
         <material name="interbotix_black"/>
@@ -221,5 +221,5 @@
         <origin rpy="0 0 ${pi/2}" xyz="-0.02 0 0"/>
         <geometry>
-          <mesh filename="package://interbotix_xsarm_descriptions/meshes/wx250_meshes/wx250_6_gripper.stl" scale="0.001 0.001 0.001"/>
+          <mesh filename="package://wx250_description/meshes/wx250_6_gripper.stl" scale="0.001 0.001 0.001"/>
         </geometry>
       </collision>
@@ -263,5 +263,5 @@
         <origin rpy="0 0 ${pi/2}" xyz="-0.0685 0 0"/>
         <geometry>
-          <mesh filename="package://interbotix_xsarm_descriptions/meshes/wx250_meshes/wx250_7_gripper_prop.stl" scale="0.001 0.001 0.001"/>
+          <mesh filename="package://wx250_description/meshes/wx250_7_gripper_prop.stl" scale="0.001 0.001 0.001"/>
         </geometry>
         <material name="interbotix_black"/>
@@ -270,5 +270,5 @@
         <origin rpy="0 0 ${pi/2}" xyz="-0.0685 0 0"/>
         <geometry>
-          <mesh filename="package://interbotix_xsarm_descriptions/meshes/wx250_meshes/wx250_7_gripper_prop.stl" scale="0.001 0.001 0.001"/>
+          <mesh filename="package://wx250_description/meshes/wx250_7_gripper_prop.stl" scale="0.001 0.001 0.001"/>
         </geometry>
       </collision>
@@ -291,5 +291,5 @@
           <origin rpy="0 0 0" xyz="0 0 0"/>
           <geometry>
-            <mesh filename="package://interbotix_xsarm_descriptions/meshes/wx250_meshes/wx250_10_ar_tag.stl" scale="0.001 0.001 0.001"/>
+            <mesh filename="package://wx250_description/meshes/wx250_10_ar_tag.stl" scale="0.001 0.001 0.001"/>
           </geometry>
           <material name="interbotix_black"/>
@@ -298,5 +298,5 @@
           <origin rpy="0 0 0" xyz="0 0 0"/>
           <geometry>
-            <mesh filename="package://interbotix_xsarm_descriptions/meshes/wx250_meshes/wx250_10_ar_tag.stl" scale="0.001 0.001 0.001"/>
+            <mesh filename="package://wx250_description/meshes/wx250_10_ar_tag.stl" scale="0.001 0.001 0.001"/>
           </geometry>
         </collision>
@@ -320,5 +320,5 @@
           <origin rpy="0 0 ${pi/2}" xyz="-0.063 0 0"/>
           <geometry>
-            <mesh filename="package://interbotix_xsarm_descriptions/meshes/wx250_meshes/wx250_8_gripper_bar.stl" scale="0.001 0.001 0.001"/>
+            <mesh filename="package://wx250_description/meshes/wx250_8_gripper_bar.stl" scale="0.001 0.001 0.001"/>
           </geometry>
           <material name="interbotix_black"/>
@@ -327,5 +327,5 @@
           <origin rpy="0 0 ${pi/2}" xyz="-0.063 0 0"/>
           <geometry>
-            <mesh filename="package://interbotix_xsarm_descriptions/meshes/wx250_meshes/wx250_8_gripper_bar.stl" scale="0.001 0.001 0.001"/>
+            <mesh filename="package://wx250_description/meshes/wx250_8_gripper_bar.stl" scale="0.001 0.001 0.001"/>
           </geometry>
         </collision>
@@ -371,5 +371,5 @@
             <origin rpy="${pi} ${pi} 0" xyz="0 0.005 0"/>
             <geometry>
-              <mesh filename="package://interbotix_xsarm_descriptions/meshes/wx250_meshes/wx250_9_gripper_finger.stl" scale="0.001 0.001 0.001"/>
+              <mesh filename="package://wx250_description/meshes/wx250_9_gripper_finger.stl" scale="0.001 0.001 0.001"/>
             </geometry>
             <material name="interbotix_black"/>
@@ -378,5 +378,5 @@
             <origin rpy="${pi} ${pi} 0" xyz="0 0.005 0"/>
             <geometry>
-              <mesh filename="package://interbotix_xsarm_descriptions/meshes/wx250_meshes/wx250_9_gripper_finger.stl" scale="0.001 0.001 0.001"/>
+              <mesh filename="package://wx250_description/meshes/wx250_9_gripper_finger.stl" scale="0.001 0.001 0.001"/>
             </geometry>
           </collision>
@@ -411,5 +411,5 @@
             <origin rpy="0 ${pi} 0" xyz="0 -0.005 0"/>
             <geometry>
-              <mesh filename="package://interbotix_xsarm_descriptions/meshes/wx250_meshes/wx250_9_gripper_finger.stl" scale="0.001 0.001 0.001"/>
+              <mesh filename="package://wx250_description/meshes/wx250_9_gripper_finger.stl" scale="0.001 0.001 0.001"/>
             </geometry>
             <material name="interbotix_black"/>
@@ -418,5 +418,5 @@
             <origin rpy="0 ${pi} 0" xyz="0 -0.005 0"/>
             <geometry>
-              <mesh filename="package://interbotix_xsarm_descriptions/meshes/wx250_meshes/wx250_9_gripper_finger.stl" scale="0.001 0.001 0.001"/>
+              <mesh filename="package://wx250_description/meshes/wx250_9_gripper_finger.stl" scale="0.001 0.001 0.001"/>
             </geometry>
           </collision>
