Commit message: Update robot.xacro

File: robots/go1_description/xacro/robot.xacro (robot description, xacro)
@@ -9,4 +9,6 @@
     <xacro:include filename="$(find go1_description)/xacro/depthCamera.xacro"/>
     <xacro:include filename="$(find go1_description)/xacro/ultraSound.xacro"/>
+    <!-- Include file for the robotic arm -->
+    <xacro:include filename="$(find wx250_description)/urdf/wx250.urdf.xacro" />
     <!-- <xacro:include filename="$(find go1_gazebo)/launch/stairs.urdf.xacro"/> -->
     <!-- <xacro:stairs stairs="15" xpos="0" ypos="0" zpos="0" /> -->
@@ -58,4 +60,12 @@
         </inertial>
     </link>
+    <!-- Add the robotic arm -->
+    <xacro:wx250_robot /> <!-- New addition -->
+    <!-- Attach the robotic arm to the trunk -->
+    <joint name="arm_to_trunk" type="fixed"> <!-- New addition -->
+        <parent link="trunk"/> <!-- Link to the quadruped's torso -->
+        <child link="arm_base_link"/> <!-- Base link of the arm -->
+        <origin xyz="0 0 0.3" rpy="0 0 0"/> <!-- Adjust position and orientation -->
+    </joint> <!-- New addition -->
     <joint name="imu_joint" type="fixed">
         <parent link="trunk"/>

Commit message: Update robot.xacro

File: robots/go1_description/xacro/robot.xacro (robot description, xacro)
@@ -62,10 +62,9 @@
     <!-- Add the robotic arm -->
     <xacro:wx250_robot /> <!-- New addition -->
-    <!-- Attach the robotic arm to the trunk -->
-    <joint name="arm_to_trunk" type="fixed"> <!-- New addition -->
-        <parent link="trunk"/> <!-- Link to the quadruped's torso -->
-        <child link="arm_base_link"/> <!-- Base link of the arm -->
-        <origin xyz="0 0 0.3" rpy="0 0 0"/> <!-- Adjust position and orientation -->
-    </joint> <!-- New addition -->
+    <joint name="arm_to_trunk" type="fixed">
+      <parent link="trunk"/> <!-- Parent link from the quadruped -->
+      <child link="wx250/base_link"/> <!-- Base link of the arm -->
+      <origin xyz="0 0 0.3" rpy="0 0 0"/> <!-- Adjust position and orientation -->
+    </joint>
     <joint name="imu_joint" type="fixed">
         <parent link="trunk"/>

Commit message: Update robot.xacro

File: robots/go1_description/xacro/robot.xacro (robot description, xacro)
@@ -65,5 +65,5 @@
       <parent link="trunk"/> <!-- Parent link from the quadruped -->
       <child link="wx250/base_link"/> <!-- Base link of the arm -->
-      <origin xyz="0 0 0.3" rpy="0 0 0"/> <!-- Adjust position and orientation -->
+      <origin xyz="0 0 0.058" rpy="0 0 0"/> <!-- Adjust position and orientation -->
     </joint>
     <joint name="imu_joint" type="fixed">
